Commit message: add base_footprint

File: dron_ws/src/rmtt_ros/rmtt_description/urdf/tello_talent.xacro (robot description, xacro)
@@ -19,4 +19,12 @@
     </material>
     <!-- TODO add Gazebo color information -->
+    <!-- Base Footprint -->
+    <link name="${tf_prefix}base_footprint"/>
+    <joint name="base_footprint_joint" type="fixed">
+        <!-- <origin xyz="0 0 0" rpy="${-pi} ${-pi*90/180} ${-pi*90/180}"/> -->
+        <origin xyz="0 0 0" rpy="0 0 0"/>
+        <parent link="${tf_prefix}base_footprint"/>
+        <child link="${tf_prefix}base_link"/>
+    </joint>
     <!-- Base link -->
     <link name="${tf_prefix}base_link">
@@ -85,5 +93,5 @@
     <!-- Fixed joint -->
     <joint name="camera_joint" type="fixed">
-        <origin xyz="0.035 0 0" rpy="${-pi*105/180} 0 ${-pi*90/180}"/>  <!-- TODO fix origin -->
+        <origin xyz="0.035 0 0" rpy="${-pi*90/180} 0 ${-pi*90/180}"/>  <!-- TODO fix origin -->
         <parent link="${tf_prefix}base_link"/>
         <child link="${tf_prefix}camera_link"/>

Commit message: add apriltag demo files

File: dron_ws/src/rmtt_ros/rmtt_description/urdf/tello_talent.xacro (robot description, xacro)
@@ -93,5 +93,6 @@
     <!-- Fixed joint -->
     <joint name="camera_joint" type="fixed">
-        <origin xyz="0.035 0 0" rpy="${-pi*90/180} 0 ${-pi*90/180}"/>  <!-- TODO fix origin -->
+        <origin xyz="0.035 0 0" rpy="${-pi*105/180} ${pi} ${-pi*90/180}"/>
+        <!-- <origin xyz="0.035 0 0" rpy="${-pi*160/180} 0 0"/> -->
         <parent link="${tf_prefix}base_link"/>
         <child link="${tf_prefix}camera_link"/>

Commit message: add Dr.HemanLab

File: dron_ws/src/rmtt_ros/rmtt_description/urdf/tello_talent.xacro (robot description, xacro)
@@ -93,6 +93,8 @@
     <!-- Fixed joint -->
     <joint name="camera_joint" type="fixed">
+        <!-- AprilTag -->
         <origin xyz="0.035 0 0" rpy="${-pi*105/180} ${pi} ${-pi*90/180}"/>
-        <!-- <origin xyz="0.035 0 0" rpy="${-pi*160/180} 0 0"/> -->
+        <!-- OrbSlam -->
+        <!-- <origin xyz="0.035 0 0" rpy="${-pi*90/180} 0 ${-pi*90/180}"/> -->
         <parent link="${tf_prefix}base_link"/>
         <child link="${tf_prefix}camera_link"/>
